Commit message: Added custom peripheral for internal project

File: annin_ar4_description/urdf/ar_macro.xacro (robot description, xacro)
@@ -239,4 +239,34 @@
       />
     </joint>
+    <!-- <joint name="${tf_prefix}camera_holder_joint" type="fixed">
+      <origin xyz="0.01104 0.025 -0.0984" rpy="0.0 -1.57 -1.57"/>
+      <parent link="${tf_prefix}link_5"/>
+      <child link="${tf_prefix}camera_holder_link"/>
+    </joint> -->
+    <joint name="${tf_prefix}camera_holder_joint" type="fixed">
+      <origin xyz="-0.025 -0.01104 -0.13135" rpy="-3.14 1.57 0.0"/>
+      <parent link="${tf_prefix}link_4"/>
+      <child link="${tf_prefix}camera_holder_link"/>
+    </joint>
+    <link name="${tf_prefix}camera_holder_link">
+      <visual>
+        <geometry>
+          <mesh filename="file://$(find annin_ar4_description)/meshes/ar4/J6_Peripheral_HolderXRealsenseD415.STL" />
+        </geometry>
+        <material name="">
+          <color rgba="1 1 0 1"/>
+        </material>
+      </visual>
+      <collision>
+        <geometry>
+          <mesh filename="file://$(find annin_ar4_description)/meshes/ar4/J6_Peripheral_HolderXRealsenseD415.STL" />
+        </geometry>
+      </collision>
+      <inertial>
+        <origin xyz="0.0 0.0 0.0"/>
+        <mass value="0.08"/>
+        <inertia ixx="0.00000002" ixy="0.00000002" ixz="0.00000002" iyy="0.00000002" iyz="0.00000002" izz="0.00000002"/>
+      </inertial>
+    </link>
     <!-- center of the end effector mounting surface on link_6 -->
     <link name="${tf_prefix}ee_link" />

File: annin_ar4_moveit_config/srdf/ar_macro.srdf.xacro (robot description, xacro)
@@ -40,4 +40,10 @@
     <disable_collisions link1="${tf_prefix}link_4" link2="${tf_prefix}link_5" reason="Adjacent" />
     <disable_collisions link1="${tf_prefix}link_5" link2="${tf_prefix}link_6" reason="Adjacent" />
+    <disable_collisions link1="${tf_prefix}camera_holder_link" link2="${tf_prefix}base_link" reason="Never" />
+    <disable_collisions link1="${tf_prefix}camera_holder_link" link2="${tf_prefix}link_1" reason="Never" />
+    <disable_collisions link1="${tf_prefix}camera_holder_link" link2="${tf_prefix}link_2" reason="Never" />
+    <disable_collisions link1="${tf_prefix}camera_holder_link" link2="${tf_prefix}link_4" reason="Adjacent" />
+    <disable_collisions link1="${tf_prefix}camera_holder_link" link2="${tf_prefix}link_5" reason="Never" />
+    <disable_collisions link1="${tf_prefix}camera_holder_link" link2="${tf_prefix}link_6" reason="Never" />
   </xacro:macro>
 </robot>

Commit message: changed to calib_sequence that allows peripherals + some cleaning

File: annin_ar4_description/urdf/ar_macro.xacro (robot description, xacro)
@@ -239,9 +239,4 @@
       />
     </joint>
-    <!-- <joint name="${tf_prefix}camera_holder_joint" type="fixed">
-      <origin xyz="0.01104 0.025 -0.0984" rpy="0.0 -1.57 -1.57"/>
-      <parent link="${tf_prefix}link_5"/>
-      <child link="${tf_prefix}camera_holder_link"/>
-    </joint> -->
     <joint name="${tf_prefix}camera_holder_joint" type="fixed">
       <origin xyz="-0.025 -0.01104 -0.13135" rpy="-3.14 1.57 0.0"/>

Commit message: small update

File: annin_ar4_description/urdf/ar_macro.xacro (robot description, xacro)
@@ -261,5 +261,5 @@
         <origin xyz="0.0 0.0 0.0"/>
         <mass value="0.08"/>
-        <inertia ixx="0.00000002" ixy="0.00000002" ixz="0.00000002" iyy="0.00000002" iyz="0.00000002" izz="0.00000002"/>
+        <inertia ixx="0.00001" ixy="0.0" ixz="0.0" iyy="0.00001" iyz="0.0" izz="0.00001"/>
       </inertial>
     </link>
